File: pcb/upico.kicad_pcb (KiCad board)
At the start: 6 copper layers, 33.5 x 77 mm, 4 parts, among them J201 uConsoleEXT, J202 Conn_02x16_Odd_Even

Commit message: speakers
Parts:
- removed J202: Conn_02x16_Odd_Even, Connector_PinSocket_2.54mm:PinSocket_2x16_P2.54mm_Vertical
- added C1: 10uF, Capacitor_SMD:C_0603_1608Metric, F.Cu at (76.1, 90.7)
- added C10: 27pF, Capacitor_SMD:C_0402_1005Metric_Pad0.74x0.62mm_HandSolder, F.Cu at (68.0, 91.4)
- added C11: 27pF, Capacitor_SMD:C_0402_1005Metric_Pad0.74x0.62mm_HandSolder, F.Cu at (68.0, 89.5)
- added C12: 10uF, Capacitor_SMD:C_0603_1608Metric, F.Cu at (72.1, 80.7)
- added C2: 10uF, Capacitor_SMD:C_0603_1608Metric, F.Cu at (76.1, 88.2)
- added C3: 10uF, Capacitor_SMD:C_0603_1608Metric, F.Cu at (76.1, 85.7)
- added C4: 100nF, Capacitor_SMD:C_0603_1608Metric, F.Cu at (76.1, 83.2)
- added C5: 100nF, Capacitor_SMD:C_0603_1608Metric, F.Cu at (76.1, 80.7)
- added C6: 100nF, Capacitor_SMD:C_0603_1608Metric, F.Cu at (72.1, 90.7)
- added C7: 10uF, Capacitor_SMD:C_0603_1608Metric, F.Cu at (72.1, 88.2)
- added C8: 10uF, Capacitor_SMD:C_0603_1608Metric, F.Cu at (72.1, 85.7)
- added C9: 10uF, Capacitor_SMD:C_0603_1608Metric, F.Cu at (72.1, 83.2)
- added J2: uPico Connect, Connector_PinSocket_2.54mm:PinSocket_2x16_P2.54mm_Horizontal, F.Cu at (80.8, 119.3)
- added J3: QWIIC, Connector_JST:JST_SH_SM04B-SRSS-TB_1x04-1MP_P1.00mm_Horizontal, F.Cu at (70.9, 128.9)
- added J4: UART INT, Connector_JST:JST_SH_SM04B-SRSS-TB_1x04-1MP_P1.00mm_Horizontal, F.Cu at (70.9, 121.3)
- added J5: USB_C, @jb:USB_C_Receptacle_JAE_DX07S016JA3R1500, F.Cu at (87.2, 72.8)
- added J6: uConsoleSpeaker, @upico:speaker, B.Cu at (71.3, 56.2)
- added J7: uConsoleSpeaker, @upico:speaker, B.Cu at (71.4, 121.1)
- added R1: 1K, Resistor_SMD:R_0402_1005Metric_Pad0.72x0.64mm_HandSolder, F.Cu at (76.5, 106.9)
- added R2: 1K, Resistor_SMD:R_0402_1005Metric_Pad0.72x0.64mm_HandSolder, F.Cu at (76.5, 104.9)
- added R3: 1K, Resistor_SMD:R_0402_1005Metric_Pad0.72x0.64mm_HandSolder, F.Cu at (76.5, 102.9)
- added R4: 1K, Resistor_SMD:R_0402_1005Metric_Pad0.72x0.64mm_HandSolder, F.Cu at (76.5, 100.9)
- added R5: 1K, Resistor_SMD:R_0402_1005Metric_Pad0.72x0.64mm_HandSolder, F.Cu at (76.5, 98.9)
- added R6: 1K, Resistor_SMD:R_0402_1005Metric_Pad0.72x0.64mm_HandSolder, F.Cu at (76.5, 97.0)
- added R7: 1K, Resistor_SMD:R_0402_1005Metric_Pad0.72x0.64mm_HandSolder, F.Cu at (76.5, 95.0)
- added R8: 1K, Resistor_SMD:R_0402_1005Metric_Pad0.72x0.64mm_HandSolder, F.Cu at (76.5, 93.0)
- added U1: AP22652_3x, Package_TO_SOT_SMD:SOT-23-6, F.Cu at (71.1, 69.8)
- added U2: AP22652_3x, Package_TO_SOT_SMD:SOT-23-6, F.Cu at (71.1, 65.4)
- added U3: AP22652_3x, Package_TO_SOT_SMD:SOT-23-6, F.Cu at (71.1, 61.0)
- added U4: RP2040, Package_DFN_QFN:QFN-56-1EP_7x7mm_P0.4mm_EP3.2x3.2mm, F.Cu at (68.8, 105.3)
- added U5: W25Q32JVZP, Package_SON:WSON-8-1EP_6x5mm_P1.27mm_EP3.4x4.3mm, F.Cu at (69.6, 97.4)
- added Y1: Crystal, Crystal:Crystal_SMD_5032-2Pin_5.0x3.2mm, F.Cu at (74.5, 77.0)
- J1: renamed from J201; footprint @upico:mini-PCIe -> @upico:uConsoleExt
Connections:
- net Net-(J202-Pin_3) renamed +5V
- net Net-(J202-Pin_5) renamed +3.3V
- J1 pad 1: Net-(J201-SPK_LP) -> unconnected-(J1-SPK_LP-Pad1)
- J1 pad 13: Net-(J201-USB4_DP) -> unconnected-(J1-USB4_DP-Pad13)
- J1 pad 14: Net-(J201-SPK_RP) -> unconnected-(J1-SPK_RP-Pad14)
- J1 pad 15: Net-(J201-USB4_DM) -> unconnected-(J1-USB4_DM-Pad15)
- J1 pad 16: Net-(J201-SPK_RN) -> unconnected-(J1-SPK_RN-Pad16)
- J1 pad 18: Net-(J201-GPIO28) -> unconnected-(J1-GPIO28-Pad18)
- J1 pad 20: Net-(J201-GPIO29) -> unconnected-(J1-GPIO29-Pad20)
- J1 pad 22: Net-(J201-GPIO30) -> unconnected-(J1-GPIO30-Pad22)
- J1 pad 24: Net-(J201-GPIO31) -> unconnected-(J1-GPIO31-Pad24)
- J1 pad 26: Net-(J201-GPIO32) -> unconnected-(J1-GPIO32-Pad26)
- J1 pad 28: Net-(J201-GPIO33) -> unconnected-(J1-GPIO33-Pad28)
- J1 pad 3: Net-(J201-SPK_LN) -> unconnected-(J1-SPK_LN-Pad3)
- J1 pad 30: Net-(J201-GPIO34) -> unconnected-(J1-GPIO34-Pad30)
- J1 pad 32: Net-(J201-GPIO35) -> unconnected-(J1-GPIO35-Pad32)
- J1 pad 34: Net-(J201-GPIO36) -> unconnected-(J1-GPIO36-Pad34)
- J1 pad 36: Net-(J201-GPIO37) -> unconnected-(J1-GPIO37-Pad36)
- J1 pad 38: Net-(J201-GPIO38) -> unconnected-(J1-GPIO38-Pad38)
- J1 pad 40: Net-(J201-GPIO39) -> unconnected-(J1-GPIO39-Pad40)
- J1 pad 42: Net-(J201-GPIO40) -> unconnected-(J1-GPIO40-Pad42)
- J1 pad 44: Net-(J201-GPIO41) -> unconnected-(J1-GPIO41-Pad44)
- J1 pad 46: Net-(J201-GPIO42) -> unconnected-(J1-GPIO42-Pad46)
- J1 pad 48: Net-(J201-GPIO43) -> unconnected-(J1-GPIO43-Pad48)
- J1 pad 50: Net-(J201-GPIO44) -> unconnected-(J1-GPIO44-Pad50)
- J1 pad 52: Net-(J201-GPIO45) -> unconnected-(J1-GPIO45-Pad52)
- J1 pad 7: Net-(J201-USB3_DP) -> unconnected-(J1-USB3_DP-Pad7)
- J1 pad 9: Net-(J201-USB3_DM) -> unconnected-(J1-USB3_DM-Pad9)
Routing:
- net Net-(J201-SPK_RP): track 57.6 -> 0.00 mm
- net +3.3V: track 61.2 -> 4.96 mm
- net Net-(J201-SPK_RN): track 50.6 -> 0.00 mm
- net Net-(J201-USB3_DP): track 36.4 -> 0.00 mm
- net Net-(J201-USB3_DM): track 31.6 -> 0.00 mm
- net Net-(J201-USB4_DM): track 31.2 -> 0.00 mm
- net Net-(J201-USB4_DP): track 30.4 -> 0.00 mm
- net Net-(J201-GPIO45): track 29.6 -> 0.00 mm
- net Net-(J201-GPIO28): track 29.1 -> 0.00 mm
- net +5V: track 41.8 -> 12.8 mm, vias 1 -> 0
- net Net-(J201-GPIO29): track 28.4 -> 0.00 mm
- net Net-(J201-GPIO30): track 27.7 -> 0.00 mm
- net Net-(J201-GPIO44): track 27.3 -> 0.00 mm
- net Net-(J201-GPIO31): track 27.0 -> 0.00 mm
- net Net-(J201-GPIO32): track 26.2 -> 0.00 mm
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- added copper zone on In1.Cu, net GND
- added copper zone on In4.Cu, net GND
- removed copper zone on B.Cu, net GND
- removed copper zone on F.Cu, net GND
Other:
- board text removed: "GND 5V 3V3 SPLP SPLN SPRP SPRN GND U3+ U3- GND U4+ U4- GND IO44 IO45"
- board text removed: "IO28 IO29 IO30 IO31 IO32 IO33 IO34 IO35 IO36 IO37 IO38 IO39 IO40 IO41 IO42 IO43"
- board text removed: "uConsole Ext. Proto rev: 0x01 https://vitaly.codes"

Commit message: basics
Parts:
- removed the J3 at (70.9, 128.9)
- added C10: 100nF, Capacitor_SMD:C_0402_1005Metric_Pad0.74x0.62mm_HandSolder, B.Cu at (75.2, 114.4)
- added C11: 100nF, Capacitor_SMD:C_0402_1005Metric_Pad0.74x0.62mm_HandSolder, B.Cu at (76.8, 114.4)
- added C12: 100nF, Capacitor_SMD:C_0402_1005Metric_Pad0.74x0.62mm_HandSolder, B.Cu at (73.5, 114.6)
- added C13: 100nF, Capacitor_SMD:C_0402_1005Metric_Pad0.74x0.62mm_HandSolder, B.Cu at (67.7, 114.6)
- added C3: 100nF, Capacitor_SMD:C_0402_1005Metric_Pad0.74x0.62mm_HandSolder, B.Cu at (73.1, 117.5)
- added C4: 100nF, Capacitor_SMD:C_0402_1005Metric_Pad0.74x0.62mm_HandSolder, B.Cu at (71.6, 117.6)
- added C5: 1uF, Capacitor_SMD:C_0402_1005Metric_Pad0.74x0.62mm_HandSolder, B.Cu at (69.9, 117.5)
- added C7: 100nF, Capacitor_SMD:C_0402_1005Metric_Pad0.74x0.62mm_HandSolder, B.Cu at (69.1, 114.6)
- added C8: 100nF, Capacitor_SMD:C_0402_1005Metric_Pad0.74x0.62mm_HandSolder, B.Cu at (70.7, 114.6)
- added C9: 100nF, Capacitor_SMD:C_0402_1005Metric_Pad0.74x0.62mm_HandSolder, B.Cu at (72.1, 114.6)
- added D1: LED, LED_SMD:LED_0603_1608Metric, F.Cu at (92.0, 80.9)
- added R10: DNP, Resistor_SMD:R_0402_1005Metric_Pad0.72x0.64mm_HandSolder, F.Cu at (77.7, 84.0)
- added R11: DNP, Resistor_SMD:R_0402_1005Metric_Pad0.72x0.64mm_HandSolder, F.Cu at (77.7, 86.0)
- added R12: DNP, Resistor_SMD:R_0402_1005Metric_Pad0.72x0.64mm_HandSolder, F.Cu at (77.7, 88.0)
- added R13: DNP, Resistor_SMD:R_0402_1005Metric_Pad0.72x0.64mm_HandSolder, F.Cu at (77.7, 89.9)
- added R14: 470R, Resistor_SMD:R_0402_1005Metric_Pad0.72x0.64mm_HandSolder, F.Cu at (91.6, 83.2)
- added R15: 56K, Resistor_SMD:R_0402_1005Metric_Pad0.72x0.64mm_HandSolder, B.Cu at (83.9, 75.3)
- added R17: 10K, Resistor_SMD:R_0402_1005Metric_Pad0.72x0.64mm_HandSolder, B.Cu at (74.6, 74.3)
- added R18: 10K, Resistor_SMD:R_0402_1005Metric_Pad0.72x0.64mm_HandSolder, B.Cu at (65.6, 73.4)
- added R19: 10K, Resistor_SMD:R_0402_1005Metric_Pad0.72x0.64mm_HandSolder, B.Cu at (65.4, 79.7)
- added R20: 10K, Resistor_SMD:R_0402_1005Metric_Pad0.72x0.64mm_HandSolder, B.Cu at (74.6, 73.1)
- added R4: 27R, Resistor_SMD:R_0402_1005Metric_Pad0.72x0.64mm_HandSolder, B.Cu at (67.2, 93.9)
- added R6: 0R, Resistor_SMD:R_0402_1005Metric_Pad0.72x0.64mm_HandSolder, F.Cu at (77.7, 95.5)
- added R7: 0R, Resistor_SMD:R_0402_1005Metric_Pad0.72x0.64mm_HandSolder, F.Cu at (77.7, 97.4)
- added R8: DNP, Resistor_SMD:R_0402_1005Metric_Pad0.72x0.64mm_HandSolder, F.Cu at (77.7, 99.4)
- added R9: DNP, Resistor_SMD:R_0402_1005Metric_Pad0.72x0.64mm_HandSolder, F.Cu at (77.7, 101.4)
- added TP1: GND, TestPoint:TestPoint_Pad_D1.0mm, F.Cu at (73.4, 101.3)
- added TP2: +3.3V, TestPoint:TestPoint_Pad_D1.0mm, F.Cu at (62.9, 90.4)
- added TP3: +5V, TestPoint:TestPoint_Pad_D1.0mm, F.Cu at (62.9, 81.5)
- added TP4: VDD EN, TestPoint:TestPoint_Pad_D1.0mm, F.Cu at (62.9, 74.6)
- added TP5: RUN, TestPoint:TestPoint_Pad_D1.0mm, F.Cu at (74.4, 99.5)
- added TP6: BOOT, TestPoint:TestPoint_Pad_D1.0mm, F.Cu at (72.3, 99.5)
- added TP7: USB D+, TestPoint:TestPoint_Pad_D1.0mm, F.Cu at (81.9, 72.3)
- added TP8: USB D-, TestPoint:TestPoint_Pad_D1.0mm, F.Cu at (81.9, 74.5)
- added U3: USBLC6-2P6, Package_TO_SOT_SMD:SOT-666, B.Cu at (77.6, 104.1)
- added U4: USBLC6-2P6, Package_TO_SOT_SMD:SOT-666, B.Cu at (81.9, 73.4)
- C1: renamed from C10; moved to B.Cu
- C14: renamed from C1; moved to B.Cu
- C15: renamed from C2; moved to B.Cu
- C16: renamed from C3; moved to B.Cu
- C17: renamed from C4; footprint Capacitor_SMD:C_0603_1608Metric -> Capacitor_SMD:C_0402_1005Metric_Pad0.74x0.62mm_HandSolder; moved to B.Cu
- C18: renamed from C5; footprint Capacitor_SMD:C_0603_1608Metric -> Capacitor_SMD:C_0402_1005Metric_Pad0.74x0.62mm_HandSolder; moved to B.Cu
- C19: renamed from C6; footprint Capacitor_SMD:C_0603_1608Metric -> Capacitor_SMD:C_0402_1005Metric_Pad0.74x0.62mm_HandSolder; moved to B.Cu
- C2: renamed from C11; moved to B.Cu
- C20: renamed from C7; moved to B.Cu
- C21: renamed from C8; moved to B.Cu
- C22: renamed from C9; moved to B.Cu
- C6: renamed from C12; value 10uF -> 1uF; footprint Capacitor_SMD:C_0603_1608Metric -> Capacitor_SMD:C_0402_1005Metric_Pad0.74x0.62mm_HandSolder; moved to B.Cu
- J2: moved to B.Cu
- J3: renamed from J5; moved to B.Cu
- J4: value UART INT -> Camera; footprint Connector_JST:JST_SH_SM04B-SRSS-TB_1x04-1MP_P1.00mm_Horizontal -> Connector_FFC-FPC:Hirose_FH12-22S-0.5SH_1x22-1MP_P0.50mm_Horizontal
- R1: renamed from R6; moved to B.Cu
- R16: renamed from R4; value 1K -> 56K; moved to B.Cu
- R2: renamed from R7; value 1K -> DNP
- R21: renamed from R2; value 1K -> 100K; moved to B.Cu
- R22: renamed from R3; value 1K -> 100K; moved to B.Cu
- R23: renamed from R1; value 1K -> 50K; moved to B.Cu
- R3: renamed from R8; moved to B.Cu
- R5: value 1K -> 27R; moved to B.Cu
- U1: renamed from U5; moved to B.Cu
- U2: renamed from U4; moved to B.Cu
- U5: renamed from U2; moved to B.Cu
- U6: renamed from U3; moved to B.Cu
- U7: renamed from U1; moved to B.Cu
- Y1: value Crystal -> 12MHz; moved to B.Cu
- moved R23 38.4 mm to (76.0, 68.5)
- moved J2 38.1 mm to (81.3, 81.3)
- moved R21 35.2 mm to (70.6, 70.2), turned to 90 degrees
- moved C6 34.4 mm to (66.0, 114.6), turned to 90 degrees
- moved Y1 34.1 mm to (69.8, 110.8), turned to 0 degrees
- moved R16 30.4 mm to (83.9, 71.5), turned to -90 degrees
- moved R22 27.1 mm to (70.6, 76.5), turned to 90 degrees
- moved C15 20.8 mm to (64.8, 70.8), turned to -90 degrees
- moved C14 19.9 mm to (73.9, 70.9), turned to -90 degrees
- moved C2 19.0 mm to (72.1, 108.0), turned to 0 degrees
- moved C1 16.6 mm to (67.9, 108.0), turned to 0 degrees
- moved U6 16.4 mm to (67.8, 77.0), turned to 0 degrees
- moved C19 16.1 mm to (63.4, 77.2), turned to -90 degrees
- moved C18 16.1 mm to (63.4, 70.8), turned to -90 degrees
- moved C20 15.7 mm to (77.5, 73.5)
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- renumbered J6 to J5, J7 to J6
Connections:
- C1 pad 1: unconnected-(C10-Pad1) -> Net-(U2-XIN)
- C1 pad 2: unconnected-(C10-Pad2) -> GND
- C15 pad 2: +3.3V -> +5V
- C18 pad 2: +3.3V -> +5V
- C2 pad 1: unconnected-(C11-Pad1) -> Net-(C2-Pad1)
- C2 pad 2: unconnected-(C11-Pad2) -> GND
- C20 pad 1: EXT_5V -> VBUS
- C21 pad 1: EXT_3V -> +5VD
- C22 pad 1: PICO_PWR -> VDD
- C6 pad 1: unconnected-(C12-Pad1) -> VDD
- C6 pad 2: unconnected-(C12-Pad2) -> GND
- J1 pad 1: unconnected-(J1-SPK_LP-Pad1) -> /SPK_LP
- J1 pad 13: unconnected-(J1-USB4_DP-Pad13) -> /PICO_USB_DP
- J1 pad 14: unconnected-(J1-SPK_RP-Pad14) -> /SPK_RP
- J1 pad 15: unconnected-(J1-USB4_DM-Pad15) -> /PICO_USB_DN
- J1 pad 16: unconnected-(J1-SPK_RN-Pad16) -> /SPK_RN
- J1 pad 18: unconnected-(J1-GPIO28-Pad18) -> Net-(J1-GPIO28)
- J1 pad 20: unconnected-(J1-GPIO29-Pad20) -> Net-(J1-GPIO29)
- J1 pad 22: unconnected-(J1-GPIO30-Pad22) -> /VBUS_FLT
- J1 pad 23: unconnected-(J1-CAM_DP3-Pad23) -> /CAM_DP3
- J1 pad 24: unconnected-(J1-GPIO31-Pad24) -> /VBUS_EN
- J1 pad 25: unconnected-(J1-CAM_DN3-Pad25) -> /CAM_DN3
- J1 pad 26: unconnected-(J1-GPIO32-Pad26) -> /UART_TX
- J1 pad 28: unconnected-(J1-GPIO33-Pad28) -> /UART_RX
- J1 pad 29: unconnected-(J1-CAM_DP2-Pad29) -> /CAM_DP2
- J1 pad 3: unconnected-(J1-SPK_LN-Pad3) -> /SPK_LN
- J1 pad 31: unconnected-(J1-CAM_DN2-Pad31) -> /CAM_DN2
- J1 pad 32: unconnected-(J1-GPIO35-Pad32) -> /VDD_FLT
- J1 pad 34: unconnected-(J1-GPIO36-Pad34) -> /VDD_EN
- J1 pad 35: unconnected-(J1-CAM_CP-Pad35) -> /CAM_CP
- J1 pad 36: unconnected-(J1-GPIO37-Pad36) -> /PICO_BOOT
- J1 pad 37: unconnected-(J1-CAM_CN-Pad37) -> /CAM_CN
- J1 pad 38: unconnected-(J1-GPIO38-Pad38) -> /PICO_RUN
- J1 pad 40: unconnected-(J1-GPIO39-Pad40) -> /EXT_5V_FLT
- J1 pad 41: unconnected-(J1-CAM_DP1-Pad41) -> /CAM_DP1
- J1 pad 42: unconnected-(J1-GPIO40-Pad42) -> /EXT_5V_EN
- J1 pad 43: unconnected-(J1-CAM_DN1-Pad43) -> /CAM_DN1
- J1 pad 46: unconnected-(J1-GPIO42-Pad46) -> /CAM_EN
- J1 pad 47: unconnected-(J1-CAM_DP0-Pad47) -> /CAM_DP0
- J1 pad 48: unconnected-(J1-GPIO43-Pad48) -> /CAM_LED
- J1 pad 49: unconnected-(J1-CAM_DN0-Pad49) -> /CAM_DN0
- J1 pad 50: unconnected-(J1-GPIO44-Pad50) -> Net-(J1-GPIO44)
- J1 pad 52: unconnected-(J1-GPIO45-Pad52) -> Net-(J1-GPIO45)
- J1 pad 7: unconnected-(J1-USB3_DP-Pad7) -> /USB_DP
- J1 pad 9: unconnected-(J1-USB3_DM-Pad9) -> /USB_DN
- J2 pad 1: unconnected-(J2-Pin_1-Pad1) -> +5VD
- J2 pad 10: unconnected-(J2-Pin_10-Pad10) -> /PICO_IO14
- J2 pad 11: unconnected-(J2-Pin_11-Pad11) -> /PICO_IO9
- J2 pad 12: unconnected-(J2-Pin_12-Pad12) -> /PICO_IO13
- J2 pad 13: unconnected-(J2-Pin_13-Pad13) -> /PICO_IO8
- J2 pad 14: unconnected-(J2-Pin_14-Pad14) -> /PICO_IO12
- J2 pad 15: unconnected-(J2-Pin_15-Pad15) -> /PICO_IO27
- J2 pad 16: unconnected-(J2-Pin_16-Pad16) -> /PICO_IO29
- J2 pad 17: unconnected-(J2-Pin_17-Pad17) -> /PICO_IO26
- J2 pad 18: unconnected-(J2-Pin_18-Pad18) -> /PICO_IO28
- J2 pad 19: unconnected-(J2-Pin_19-Pad19) -> Net-(J2-Pin_19)
- J2 pad 2: unconnected-(J2-Pin_2-Pad2) -> +5VD
- J2 pad 20: unconnected-(J2-Pin_20-Pad20) -> Net-(J2-Pin_20)
- J2 pad 21: unconnected-(J2-Pin_21-Pad21) -> VDD
- J2 pad 22: unconnected-(J2-Pin_22-Pad22) -> VDD
- J2 pad 23: unconnected-(J2-Pin_23-Pad23) -> GND
- J2 pad 24: unconnected-(J2-Pin_24-Pad24) -> GND
- J2 pad 25: unconnected-(J2-Pin_25-Pad25) -> /PICO_IO3
- J2 pad 26: unconnected-(J2-Pin_26-Pad26) -> /PICO_IO7
- J2 pad 27: unconnected-(J2-Pin_27-Pad27) -> /PICO_IO2
- J2 pad 28: unconnected-(J2-Pin_28-Pad28) -> /PICO_IO6
- J2 pad 29: unconnected-(J2-Pin_29-Pad29) -> /PICO_IO1
- J2 pad 3: unconnected-(J2-Pin_3-Pad3) -> VDD
- J2 pad 30: unconnected-(J2-Pin_30-Pad30) -> /PICO_IO5
- J2 pad 31: unconnected-(J2-Pin_31-Pad31) -> /PICO_IO0
- J2 pad 32: unconnected-(J2-Pin_32-Pad32) -> /PICO_IO4
- J2 pad 4: unconnected-(J2-Pin_4-Pad4) -> VDD
- J2 pad 5: unconnected-(J2-Pin_5-Pad5) -> GND
- J2 pad 6: unconnected-(J2-Pin_6-Pad6) -> GND
- J2 pad 7: unconnected-(J2-Pin_7-Pad7) -> /PICO_IO11
- J2 pad 8: unconnected-(J2-Pin_8-Pad8) -> /PICO_IO15
- J2 pad 9: unconnected-(J2-Pin_9-Pad9) -> /PICO_IO10
- J3 pad A1: unconnected-(J5-GND-PadA1) -> GND
- J3 pad A4: Net-(J5-VBUS-PadA4) -> VBUS
- J3 pad A5: unconnected-(J5-CC1-PadA5) -> Net-(J3-CC1)
- J3 pad A6: unconnected-(J5-D+-PadA6) -> Net-(J3-D+-PadA6)
- J3 pad A7: unconnected-(J5-D--PadA7) -> Net-(J3-D--PadA7)
- J3 pad A9: Net-(J5-VBUS-PadA4) -> VBUS
- J3 pad B5: unconnected-(J5-CC2-PadB5) -> Net-(J3-CC2)
- J3 pad B6: unconnected-(J5-D+-PadB6) -> Net-(J3-D+-PadA6)
- J3 pad B7: unconnected-(J5-D--PadB7) -> Net-(J3-D--PadA7)
- J4 pad 1: unconnected-(J4-Pin_1-Pad1) -> GND
- J4 pad 2: unconnected-(J4-Pin_2-Pad2) -> /CAM_DN0
- J4 pad 3: unconnected-(J4-Pin_3-Pad3) -> /CAM_DP0
- J4 pad 4: unconnected-(J4-Pin_4-Pad4) -> GND
- J5 pad 1: unconnected-(J6-P1-Pad1) -> /SPK_LP
- J5 pad 2: unconnected-(J6-N1-Pad2) -> /SPK_LN
- J5 pad 3: unconnected-(J6-P2-Pad3) -> /SPK_LP
- J5 pad 4: unconnected-(J6-N2-Pad4) -> /SPK_LN
- J6 pad 1: unconnected-(J7-P1-Pad1) -> /SPK_RP
- J6 pad 2: unconnected-(J7-N1-Pad2) -> /SPK_RN
- J6 pad 3: unconnected-(J7-P2-Pad3) -> /SPK_RP
- J6 pad 4: unconnected-(J7-N2-Pad4) -> /SPK_RN
- R1 pad 1: unconnected-(R6-Pad1) -> /PICO_BOOT
- R1 pad 2: unconnected-(R6-Pad2) -> Net-(U1-~{CS})
- R16 pad 1: unconnected-(R4-Pad1) -> VBUS
- R16 pad 2: unconnected-(R4-Pad2) -> Net-(J3-CC1)
- R2 pad 1: unconnected-(R7-Pad1) -> VDD
- R2 pad 2: unconnected-(R7-Pad2) -> Net-(U1-~{CS})
- R3 pad 1: unconnected-(R8-Pad1) -> Net-(C2-Pad1)
- R3 pad 2: unconnected-(R8-Pad2) -> Net-(U2-XOUT)
- R5 pad 1: unconnected-(R5-Pad1) -> /PICO_USB_DN
- R5 pad 2: unconnected-(R5-Pad2) -> Net-(U2-USB_DM)
- U1 pad 1: unconnected-(U5-~{CS}-Pad1) -> Net-(U1-~{CS})
- U1 pad 2: unconnected-(U5-DO(IO1)-Pad2) -> Net-(U1-DO(IO1))
- U1 pad 3: unconnected-(U5-IO2-Pad3) -> Net-(U1-IO2)
- U1 pad 4: unconnected-(U5-GND-Pad4) -> GND
- U1 pad 5: unconnected-(U5-DI(IO0)-Pad5) -> Net-(U1-DI(IO0))
- U1 pad 6: unconnected-(U5-CLK-Pad6) -> Net-(U1-CLK)
- U1 pad 7: unconnected-(U5-IO3-Pad7) -> Net-(U1-IO3)
- U1 pad 8: unconnected-(U5-VCC-Pad8) -> VDD
- U1 pad 9: unconnected-(U5-EP-Pad9) -> GND
- U2 pad 1: Net-(U4-IOVDD-Pad1) -> VDD
- U2 pad 10: Net-(U4-IOVDD-Pad1) -> VDD
- U2 pad 11: unconnected-(U4-GPIO8-Pad11) -> /PICO_IO8
- U2 pad 12: unconnected-(U4-GPIO9-Pad12) -> /PICO_IO9
- U2 pad 13: unconnected-(U4-GPIO10-Pad13) -> /PICO_IO10
- U2 pad 14: unconnected-(U4-GPIO11-Pad14) -> /PICO_IO11
- U2 pad 15: unconnected-(U4-GPIO12-Pad15) -> /PICO_IO12
- U2 pad 16: unconnected-(U4-GPIO13-Pad16) -> /PICO_IO13
- U2 pad 17: unconnected-(U4-GPIO14-Pad17) -> /PICO_IO14
- U2 pad 18: unconnected-(U4-GPIO15-Pad18) -> /PICO_IO15
- U2 pad 19: unconnected-(U4-TESTEN-Pad19) -> GND
- U2 pad 2: unconnected-(U4-GPIO0-Pad2) -> /PICO_IO0
- U2 pad 20: unconnected-(U4-XIN-Pad20) -> Net-(U2-XIN)
- U2 pad 21: unconnected-(U4-XOUT-Pad21) -> Net-(U2-XOUT)
- U2 pad 22: Net-(U4-IOVDD-Pad1) -> VDD
- U2 pad 23: Net-(U4-DVDD-Pad23) -> Net-(U2-VREG_VOUT)
- U2 pad 26: unconnected-(U4-RUN-Pad26) -> /PICO_RUN
- U2 pad 27: unconnected-(U4-GPIO16-Pad27) -> Net-(U2-GPIO16)
- U2 pad 28: unconnected-(U4-GPIO17-Pad28) -> Net-(U2-GPIO17)
- U2 pad 3: unconnected-(U4-GPIO1-Pad3) -> /PICO_IO1
- U2 pad 31: unconnected-(U4-GPIO20-Pad31) -> Net-(U2-GPIO20)
- U2 pad 32: unconnected-(U4-GPIO21-Pad32) -> Net-(U2-GPIO21)
- U2 pad 33: Net-(U4-IOVDD-Pad1) -> VDD
- U2 pad 37: unconnected-(U4-GPIO25-Pad37) -> /LED
- U2 pad 38: unconnected-(U4-GPIO26_ADC0-Pad38) -> /PICO_IO27
- U2 pad 39: unconnected-(U4-GPIO27_ADC1-Pad39) -> /PICO_IO26
- U2 pad 4: unconnected-(U4-GPIO2-Pad4) -> /PICO_IO2
- U2 pad 40: unconnected-(U4-GPIO28_ADC2-Pad40) -> /PICO_IO28
- U2 pad 41: unconnected-(U4-GPIO29_ADC3-Pad41) -> /PICO_IO29
- U2 pad 42: Net-(U4-IOVDD-Pad1) -> VDD
- U2 pad 43: unconnected-(U4-ADC_AVDD-Pad43) -> VDD
- U2 pad 44: unconnected-(U4-VREG_IN-Pad44) -> VDD
- U2 pad 45: unconnected-(U4-VREG_VOUT-Pad45) -> Net-(U2-VREG_VOUT)
- U2 pad 46: unconnected-(U4-USB_DM-Pad46) -> Net-(U2-USB_DM)
- U2 pad 47: unconnected-(U4-USB_DP-Pad47) -> Net-(U2-USB_DP)
- U2 pad 48: unconnected-(U4-USB_VDD-Pad48) -> VDD
- U2 pad 49: Net-(U4-IOVDD-Pad1) -> VDD
- U2 pad 5: unconnected-(U4-GPIO3-Pad5) -> /PICO_IO3
- U2 pad 50: Net-(U4-DVDD-Pad23) -> Net-(U2-VREG_VOUT)
- U2 pad 51: unconnected-(U4-QSPI_SD3-Pad51) -> Net-(U1-IO3)
- U2 pad 52: unconnected-(U4-QSPI_SCLK-Pad52) -> Net-(U1-CLK)
- U2 pad 53: unconnected-(U4-QSPI_SD0-Pad53) -> Net-(U1-DI(IO0))
- U2 pad 54: unconnected-(U4-QSPI_SD2-Pad54) -> Net-(U1-IO2)
- U2 pad 55: unconnected-(U4-QSPI_SD1-Pad55) -> Net-(U1-DO(IO1))
- U2 pad 56: unconnected-(U4-QSPI_SS-Pad56) -> Net-(U1-~{CS})
- U2 pad 57: unconnected-(U4-GND-Pad57) -> GND
- U2 pad 6: unconnected-(U4-GPIO4-Pad6) -> /PICO_IO4
- U2 pad 7: unconnected-(U4-GPIO5-Pad7) -> /PICO_IO5
- U2 pad 8: unconnected-(U4-GPIO6-Pad8) -> /PICO_IO6
- U2 pad 9: unconnected-(U4-GPIO7-Pad9) -> /PICO_IO7
- U5 pad 1: +3.3V -> +5V
- U5 pad 3: EXT_3V_EN -> /EXT_5V_EN
- U5 pad 4: EXT_3V_FLT -> /EXT_5V_FLT
- U5 pad 6: EXT_3V -> +5VD
- U6 pad 3: PICO_PWR_EN -> /VDD_EN
- U6 pad 4: PICO_PWR_FLT -> /VDD_FLT
- U6 pad 6: PICO_PWR -> VDD
- U7 pad 3: EXT_5V_EN -> /VBUS_EN
- U7 pad 4: EXT_5V_FLT -> /VBUS_FLT
- U7 pad 6: EXT_5V -> VBUS
- Y1 pad 1: unconnected-(Y1-Pad1) -> Net-(U2-XIN)
- Y1 pad 2: unconnected-(Y1-Pad2) -> Net-(C2-Pad1)
Routing:
- net /SPK_RP: track 0.00 -> 71.6 mm, vias 0 -> 2
- net /SPK_RN: track 0.00 -> 67.1 mm, vias 0 -> 2
- net +3.3V: track 4.96 -> 70.5 mm, vias 0 -> 4
- net /SPK_LP: track 0.00 -> 46.1 mm, vias 0 -> 2
- net /SPK_LN: track 0.00 -> 45.0 mm, vias 0 -> 2
- net /CAM_DP3: track 0.00 -> 37.2 mm
- net /CAM_DN3: track 0.00 -> 36.4 mm
- net /CAM_DP2: track 0.00 -> 35.4 mm
- net /CAM_DN2: track 0.00 -> 34.6 mm
- net /CAM_CP: track 0.00 -> 31.1 mm
- net /CAM_CN: track 0.00 -> 30.4 mm
- net /CAM_DP1: track 0.00 -> 28.2 mm
- net /CAM_DN1: track 0.00 -> 27.4 mm
- net /CAM_DP0: track 0.00 -> 25.2 mm
- net /CAM_DN0: track 0.00 -> 24.4 mm
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- added copper zone on B.Cu, net +5V
- added copper zone on In2.Cu, net VDD

Commit message: aux routing
Parts:
- added R15: DNP, Resistor_SMD:R_0402_1005Metric, F.Cu at (61.4, 115.6)
- added R16: DNP, Resistor_SMD:R_0402_1005Metric, F.Cu at (61.4, 114.5)
- C1, C10, C11, C12, C13, C17, C18, C19, C2, C3, C4, C5, C6, C7, C8, C9: footprint Capacitor_SMD:C_0402_1005Metric_Pad0.74x0.62mm_HandSolder -> Capacitor_SMD:C_0402_1005Metric
- D1: footprint LED_SMD:LED_0603_1608Metric -> LED_THT:LED_SideEmitter_Rectangular_W4.5mm_H1.6mm; moved to B.Cu
- J1: footprint @upico:uConsoleExt -> @upico:ext
- R1, R2, R3, R4, R5, R8, R9: footprint Resistor_SMD:R_0402_1005Metric_Pad0.72x0.64mm_HandSolder -> Resistor_SMD:R_0402_1005Metric
- R10, R11: value DNP -> 2.2K; footprint Resistor_SMD:R_0402_1005Metric_Pad0.72x0.64mm_HandSolder -> Resistor_SMD:R_0402_1005Metric
- R12: renamed from R14; footprint Resistor_SMD:R_0402_1005Metric_Pad0.72x0.64mm_HandSolder -> Resistor_SMD:R_0402_1005Metric; moved to B.Cu
- R13: renamed from R12; footprint Resistor_SMD:R_0402_1005Metric_Pad0.72x0.64mm_HandSolder -> Resistor_SMD:R_0402_1005Metric
- R14: renamed from R13; footprint Resistor_SMD:R_0402_1005Metric_Pad0.72x0.64mm_HandSolder -> Resistor_SMD:R_0402_1005Metric
- R17: renamed from R15; footprint Resistor_SMD:R_0402_1005Metric_Pad0.72x0.64mm_HandSolder -> Resistor_SMD:R_0402_1005Metric
- R18: renamed from R16; footprint Resistor_SMD:R_0402_1005Metric_Pad0.72x0.64mm_HandSolder -> Resistor_SMD:R_0402_1005Metric
- R19: renamed from R17; footprint Resistor_SMD:R_0402_1005Metric_Pad0.72x0.64mm_HandSolder -> Resistor_SMD:R_0402_1005Metric
- R20: renamed from R18; footprint Resistor_SMD:R_0402_1005Metric_Pad0.72x0.64mm_HandSolder -> Resistor_SMD:R_0402_1005Metric
- R21: renamed from R19; footprint Resistor_SMD:R_0402_1005Metric_Pad0.72x0.64mm_HandSolder -> Resistor_SMD:R_0402_1005Metric
- R22: renamed from R20; footprint Resistor_SMD:R_0402_1005Metric_Pad0.72x0.64mm_HandSolder -> Resistor_SMD:R_0402_1005Metric
- R23: renamed from R21; footprint Resistor_SMD:R_0402_1005Metric_Pad0.72x0.64mm_HandSolder -> Resistor_SMD:R_0402_1005Metric
- R24: renamed from R22; footprint Resistor_SMD:R_0402_1005Metric_Pad0.72x0.64mm_HandSolder -> Resistor_SMD:R_0402_1005Metric
- R25: renamed from R23; footprint Resistor_SMD:R_0402_1005Metric_Pad0.72x0.64mm_HandSolder -> Resistor_SMD:R_0402_1005Metric
- R6, R7: value 0R -> 200R; footprint Resistor_SMD:R_0402_1005Metric_Pad0.72x0.64mm_HandSolder -> Resistor_SMD:R_0402_1005Metric
- U1: value W25Q32JVZP -> W25Q32JV; footprint Package_SON:WSON-8-1EP_6x5mm_P1.27mm_EP3.4x4.3mm -> @upico:USON-8_4x3mm_P0.8mm
- moved R10 39.6 mm to (61.4, 120.0), turned to 180 degrees
- moved R11 38.8 mm to (61.4, 121.2), turned to 180 degrees
- moved R12 33.8 mm to (63.4, 101.9), turned to 180 degrees
- moved R6 28.1 mm to (61.4, 118.4), turned to 180 degrees
- moved R13 26.5 mm to (62.3, 109.5), turned to 90 degrees
- moved R7 25.6 mm to (61.4, 117.2), turned to 180 degrees
- moved R14 25.6 mm to (61.2, 109.5), turned to 90 degrees
- moved TP7 24.7 mm to (68.6, 93.1), turned to -90 degrees
- moved TP8 24.2 mm to (66.4, 93.1), turned to -90 degrees
- moved C4 22.3 mm to (65.5, 96.0), turned to 90 degrees
- moved C10 21.2 mm to (64.0, 96.5), turned to 180 degrees
- moved R8 21.2 mm to (61.4, 113.0)
- moved C5 20.6 mm to (66.7, 97.2), turned to 90 degrees
- moved R9 19.4 mm to (61.4, 111.8)
- moved C11 19.2 mm to (68.4, 97.2), turned to 90 degrees
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Connections:
- D1 pad 1: /LED -> Net-(D1-K)
- D1 pad 2: Net-(D1-A) -> VDD
- R10 pad 1: Net-(U2-GPIO16) -> +3.3V
- R10 pad 2: /I2C_SDA -> /I2C_SCL
- R11 pad 1: Net-(U2-GPIO17) -> +3.3V
- R11 pad 2: /I2C_SCL -> /I2C_SDA
- R12 pad 1: Net-(D1-A) -> Net-(U2-GPIO25)
- R12 pad 2: VDD -> Net-(D1-K)
- R13 pad 1: Net-(U2-GPIO20) -> Net-(U2-GPIO16)
- R14 pad 1: Net-(U2-GPIO21) -> Net-(U2-GPIO17)
- U2 pad 29: unconnected-(U2-GPIO18-Pad29) -> Net-(U2-GPIO18)
- U2 pad 30: unconnected-(U2-GPIO19-Pad30) -> Net-(U2-GPIO19)
- U2 pad 31: Net-(U2-GPIO20) -> unconnected-(U2-GPIO20-Pad31)
- U2 pad 32: Net-(U2-GPIO21) -> unconnected-(U2-GPIO21-Pad32)
- U2 pad 37: /LED -> Net-(U2-GPIO25)
Routing:
- net /I2C_SCL: track 0.00 -> 49.9 mm, vias 0 -> 2
- net /I2C_SDA: track 0.00 -> 43.2 mm, vias 0 -> 2
- net /PICO_RUN: track 4.15 -> 35.9 mm, vias 0 -> 3
- net Net-(J1-GPIO28): track 5.48 -> 33.5 mm, vias 1 -> 2
- net Net-(J1-GPIO29): track 5.08 -> 30.6 mm, vias 1 -> 2
- net /PICO_BOOT: track 4.35 -> 25.0 mm, vias 0 -> 3
- net Net-(U2-GPIO17): track 0.00 -> 20.5 mm, vias 0 -> 1
- net Net-(D1-K): track 0.00 -> 20.2 mm, vias 0 -> 1
- net /EXT_5V_FLT: track 4.01 -> 22.0 mm
- net VDD: track 0.00 -> 17.9 mm, vias 0 -> 9
- net /CAM_EN: track 23.2 -> 41.0 mm, vias 1 -> 2
- net /VDD_FLT: track 4.03 -> 21.6 mm
- net GND: track 35.7 -> 53.3 mm, vias 16 -> 37
- net /EXT_5V_EN: track 4.23 -> 21.7 mm
- net /CAM_LED: track 22.9 -> 40.0 mm, vias 1 -> 2
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- added copper zone on B.Cu, net GND

Commit message: power routing
Parts:
- added C14: 10uF, Capacitor_SMD:C_0603_1608Metric, B.Cu at (82.6, 68.8)
- C5, C6: value 1uF -> 4.7uF
- R12: value 470R -> 510R
- R25: value 50K -> 47K
- moved R24 3.48 mm to (69.2, 79.0), turned to 0 degrees
- moved C23 3.41 mm to (71.1, 76.7), turned to 90 degrees
- moved C21 2.91 mm to (80.5, 71.6), turned to 0 degrees
- moved R19 1.77 mm to (73.5, 73.0), turned to 180 degrees
- moved R21 1.02 mm to (66.9, 79.0)
- moved C18 1.00 mm to (72.2, 71.1)
- moved R20 0.90 mm to (66.9, 73.0)
- moved U7 0.83 mm to (76.7, 70.6)
- moved C15 0.83 mm to (73.7, 70.8)
- moved R25 0.78 mm to (79.5, 69.8)
- moved R23 0.71 mm to (70.8, 69.8)
- moved TP6 0.69 mm to (70.3, 90.4)
- moved TP5 0.69 mm to (72.6, 90.4)
- moved C22 0.62 mm to (69.6, 73.3), turned to 0 degrees
- moved R22 0.62 mm to (75.6, 73.0)
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- renumbered C14 to C15, C15 to C16, C16 to C17, C17 to C18, C18 to C19, C19 to C20, C20 to C21, C21 to C22, C22 to C23
Routing:
- net +3.3V: track 70.4 -> 97.1 mm, vias 5 -> 6
- net /VBUS_FLT: track 17.1 -> 43.3 mm, vias 0 -> 2
- net /VBUS_EN: track 17.4 -> 42.8 mm, vias 0 -> 2
- net /EXT_5V_FLT: track 22.0 -> 43.3 mm, vias 0 -> 2
- net /EXT_5V_EN: track 21.7 -> 42.1 mm, vias 0 -> 2
- net +5V: track 11.0 -> 28.6 mm, vias 1 -> 5
- net Net-(D1-K): track 20.2 -> 4.57 mm
- net /VDD_EN: track 18.5 -> 31.2 mm, vias 1 -> 2
- net GND: track 53.3 -> 65.5 mm, vias 37 -> 52
- net VBUS: track 11.1 -> 22.6 mm
- net +5VD: track 0.00 -> 9.67 mm, vias 0 -> 1
- net /VDD_FLT: track 21.6 -> 30.3 mm
- net /PICO_IO6: track 1.68 -> 8.65 mm
- net /PICO_IO5: track 2.24 -> 6.69 mm
- net Net-(U6-ILIM): track 0.00 -> 3.40 mm
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Other:
- outline, holes or cut-outs redrawn

Commit message: control app
Parts:
- added REF**: OSHW-Logo_7.5x8mm_SilkScreen, Symbol:OSHW-Logo_7.5x8mm_SilkScreen, F.Cu at (71.1, 63.7)
- H1, H2: footprint MountingHole:MountingHole_2.7mm_M2.5_Pad_Via -> MountingHole:MountingHole_5.3mm_M5
- R2: moved to B.Cu
- R6, R7: value 200R -> DNP
- moved R2 2.54 mm to (74.9, 92.0), turned to -90 degrees
- moved D1 2.37 mm to (83.0, 79.0), turned to 180 degrees
- moved C14 0.69 mm to (82.9, 69.4), turned to 0 degrees
- moved J2 0.50 mm to (81.5, 82.2)
- moved J5 0.42 mm to (70.9, 56.2)
- moved J3 0.17 mm to (87.2, 73.8)
- moved U3 0.14 mm to (78.0, 120.1)
- moved TP7 0.14 mm to (68.5, 93.1)
- moved TP8 0.10 mm to (66.5, 93.1)
Connections:
- D1 pad 1: Net-(D1-K) -> GND
- D1 pad 2: VDD -> Net-(D1-A)
- J2 pad 10: /PICO_IO14 -> /PICO_IO2
- J2 pad 11: /PICO_IO9 -> /PICO_IO5
- J2 pad 12: /PICO_IO13 -> /PICO_IO1
- J2 pad 13: /PICO_IO8 -> /PICO_IO4
- J2 pad 14: /PICO_IO12 -> /PICO_IO0
- J2 pad 15: /PICO_IO27 -> /PICO_IO29
- J2 pad 16: /PICO_IO29 -> /PICO_IO27
- J2 pad 17: /PICO_IO26 -> /PICO_IO28
- J2 pad 18: /PICO_IO28 -> /PICO_IO26
- J2 pad 25: /PICO_IO3 -> /PICO_IO15
- J2 pad 26: /PICO_IO7 -> /PICO_IO11
- J2 pad 27: /PICO_IO2 -> /PICO_IO14
- J2 pad 28: /PICO_IO6 -> /PICO_IO10
- J2 pad 29: /PICO_IO1 -> /PICO_IO13
- J2 pad 30: /PICO_IO5 -> /PICO_IO9
- J2 pad 31: /PICO_IO0 -> /PICO_IO12
- J2 pad 32: /PICO_IO4 -> /PICO_IO8
- J2 pad 7: /PICO_IO11 -> /PICO_IO7
- J2 pad 8: /PICO_IO15 -> /PICO_IO3
- J2 pad 9: /PICO_IO10 -> /PICO_IO6
- R12 pad 2: Net-(D1-K) -> Net-(D1-A)
- U3 pad 4: Net-(J2-Pin_19) -> Net-(J2-Pin_20)
- U3 pad 6: Net-(J2-Pin_20) -> Net-(J2-Pin_19)
Routing:
- net Net-(D1-A): track 0.00 -> 33.8 mm, vias 0 -> 1
- net /PICO_IO7: track 2.44 -> 33.9 mm
- net /PICO_IO8: track 2.48 -> 29.8 mm
- net /PICO_IO9: track 2.41 -> 24.9 mm
- net /PICO_IO3: track 1.46 -> 22.9 mm
- net /PICO_IO12: track 0.87 -> 22.3 mm
- net Net-(J2-Pin_20): track 0.00 -> 21.3 mm, vias 0 -> 1
- net /PICO_IO2: track 1.44 -> 20.3 mm
- net /PICO_IO10: track 2.27 -> 20.0 mm
- net /PICO_IO13: track 1.15 -> 18.5 mm
- net Net-(J2-Pin_19): track 0.00 -> 16.8 mm, vias 0 -> 1
- net /PICO_IO27: track 9.18 -> 25.8 mm
- net /PICO_IO1: track 1.77 -> 18.0 mm, vias 0 -> 1
- net /PICO_IO14: track 1.37 -> 17.2 mm, vias 0 -> 1
- net /PICO_IO11: track 2.21 -> 16.9 mm
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Other:
- outline, holes or cut-outs redrawn
- rule pad_to_mask_clearance: 0.0508 -> 0
- board text added: "+3.3V"
- board text added: "+5V"
- board text added: "-USB+"
- board text added: "A-04/06"
- board text added: "BOOT"
- board text added: "Camera"
- board text added: "GND"
- board text added: "I2C"
- board text added: "Pullups"
- board text added: "R-01"
- board text added: "RP2040"
- board text added: "RP2040 UART"
- board text added: "RUN"
- board text added: "VDD_EN"
- board text added: "https://bitaly.codes/upico rev: 0x01"
