File: pcb/upico.kicad_pcb (KiCad board)
At the start: 6 copper layers, 33.5 x 77 mm, 72 parts, among them J1 uConsoleEXT, J2 uPico Connect, J3 USB_C_Receptacle_USB2.0, J4 Camera, J5 uConsoleSpeaker, J6 uConsoleSpeaker, U1 W25Q32JV, U2 RP2040, U3 USBLC6-2P6, U4 USBLC6-2P6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

Commit message: update pcb
Parts:
- U1: value W25Q32JV -> W25Q32JVUX; footprint @upico:USON-8_4x3mm_P0.8mm -> @upico:USON-8_2x3mm_P0.5mm
- moved U1 0.18 mm to (71.7, 95.7)
Routing:
- net GND: track 71.5 -> 70.0 mm, vias 54 -> 53
- net Net-(U1-DO(IO1)): track 3.01 -> 2.24 mm

Commit message: fix typo
Other:
- board text added: "R01/CM4"
- board text removed: "R01/CM3"
Changed lines of the file:
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@@
     (effects (font (size 0.8 0.8) (thickness 0.15) bold) (justify left bottom))
   )
-  (gr_text "R01/CM3" (at 62.9666 118.3386) (layer "F.SilkS" knockout)
+  (gr_text "R01/CM4" (at 62.9666 118.3386) (layer "F.SilkS" knockout)
     (effects (font (size 0.8 0.8) (thickness 0.15) bold) (justify left bottom))
   )
