File: pcb/upico.kicad_pcb (KiCad board)
At the start: 6 copper layers, 33.5 x 77 mm, 72 parts, among them J1 uConsoleEXT, J2 uPico Connect, J3 USB_C_Receptacle_USB2.0, J4 Camera, J5 uConsoleSpeaker, J6 uConsoleSpeaker, U1 W25Q32JVUX, U2 RP2040, U3 USBLC6-2P6, U4 USBLC6-2P6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

Commit message: shell completions
Other:
- board text added: "CM4"
- board text added: "R01"
- board text removed: "A04/A06"
- board text removed: "R01/CM4"
Changed lines of the file:
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@@
 		)
 	)
-	(gr_text "A04/A06   "
+	(gr_text "CM4"
 		(at 62.970156 113.09376 0)
 		(layer "F.SilkS" knockout)
@@
 		)
 	)
-	(gr_text "R01/CM4"
+	(gr_text "R01"
 		(at 62.9666 118.3386 0)
 		(layer "F.SilkS" knockout)
