File: pcb/upico.kicad_sch (KiCad schematic)
At the start: 34 parts, among them J2 uPico Connect, J201 uConsoleEXT, J202 Conn_02x16_Odd_Even, J3 QWIIC, J4 UART INT, J5 USB_C, U1 AP22652_3x, U2 AP22652_3x, U3 AP22652_3x, U4 RP2040, U5 W25Q32JVZP, Y1 Crystal

Commit message: speakers
Parts:
- removed J202: Conn_02x16_Odd_Even, Connector_PinSocket_2.54mm:PinSocket_2x16_P2.54mm_Vertical, symbol Connector_Generic:Conn_02x16_Odd_Even
- added J6, J7: uConsoleSpeaker, @upico:speaker, symbol @upico:uConsoleSpeaker
- J1: renamed from J201; footprint @upico:mini-PCIe -> @upico:uConsoleExt; symbol @upico:uConsole-ext -> @upico:uConsoleExt
Connections:
- net +3.3V: now also J1.17 (3V3), J1.19 (3V3)
- net +5V: now also J1.10 (5V), J1.2 (5V), J1.4 (5V), J1.6 (5V), J1.8 (5V)

Commit message: basics
Parts:
- removed J3: QWIIC, Connector_JST:JST_SH_SM04B-SRSS-TB_1x04-1MP_P1.00mm_Horizontal, symbol Connector_Generic:Conn_01x04
- removed J4: UART INT, Connector_JST:JST_SH_SM04B-SRSS-TB_1x04-1MP_P1.00mm_Horizontal, symbol Connector_Generic:Conn_01x04
- added C10, C11, C12, C13, C3, C4, C7, C8, C9: 100nF, Capacitor_SMD:C_0402_1005Metric_Pad0.74x0.62mm_HandSolder, symbol Device:C
- added C5: 1uF, Capacitor_SMD:C_0402_1005Metric_Pad0.74x0.62mm_HandSolder, symbol Device:C
- added D1: LED, LED_SMD:LED_0603_1608Metric, symbol Device:LED
- added J4: Camera, Connector_FFC-FPC:Hirose_FH12-22S-0.5SH_1x22-1MP_P0.50mm_Horizontal, symbol Connector_Generic:Conn_01x22
- added R10, R11, R12, R13, R8, R9: DNP, Resistor_SMD:R_0402_1005Metric_Pad0.72x0.64mm_HandSolder, symbol Device:R
- added R14: 470R, Resistor_SMD:R_0402_1005Metric_Pad0.72x0.64mm_HandSolder, symbol Device:R
- added R15: 56K, Resistor_SMD:R_0402_1005Metric_Pad0.72x0.64mm_HandSolder, symbol Device:R
- added R17, R18, R19, R20: 10K, Resistor_SMD:R_0402_1005Metric_Pad0.72x0.64mm_HandSolder, symbol Device:R
- added R4: 27R, Resistor_SMD:R_0402_1005Metric_Pad0.72x0.64mm_HandSolder, symbol Device:R
- added R6, R7: 0R, Resistor_SMD:R_0402_1005Metric_Pad0.72x0.64mm_HandSolder, symbol Device:R
- added TP1: GND, TestPoint:TestPoint_Pad_D1.0mm, symbol Connector:TestPoint
- added TP2: +3.3V, TestPoint:TestPoint_Pad_D1.0mm, symbol Connector:TestPoint
- added TP3: +5V, TestPoint:TestPoint_Pad_D1.0mm, symbol Connector:TestPoint
- added TP4: VDD EN, TestPoint:TestPoint_Pad_D1.0mm, symbol Connector:TestPoint
- added TP5: RUN, TestPoint:TestPoint_Pad_D1.0mm, symbol Connector:TestPoint
- added TP6: BOOT, TestPoint:TestPoint_Pad_D1.0mm, symbol Connector:TestPoint
- added TP7: USB D+, TestPoint:TestPoint_Pad_D1.0mm, symbol Connector:TestPoint
- added TP8: USB D-, TestPoint:TestPoint_Pad_D1.0mm, symbol Connector:TestPoint
- added U3, U4: USBLC6-2P6, Package_TO_SOT_SMD:SOT-666, symbol Power_Protection:USBLC6-2P6
- C17: renamed from C4; footprint Capacitor_SMD:C_0603_1608Metric -> Capacitor_SMD:C_0402_1005Metric_Pad0.74x0.62mm_HandSolder
- C18: renamed from C5; footprint Capacitor_SMD:C_0603_1608Metric -> Capacitor_SMD:C_0402_1005Metric_Pad0.74x0.62mm_HandSolder
- C19: renamed from C6; footprint Capacitor_SMD:C_0603_1608Metric -> Capacitor_SMD:C_0402_1005Metric_Pad0.74x0.62mm_HandSolder
- C6: renamed from C12; value 10uF -> 1uF; footprint Capacitor_SMD:C_0603_1608Metric -> Capacitor_SMD:C_0402_1005Metric_Pad0.74x0.62mm_HandSolder
- R16: renamed from R4; value 1K -> 56K
- R2: renamed from R7; value 1K -> DNP
- R21: renamed from R2; value 1K -> 100K
- R22: renamed from R3; value 1K -> 100K
- R23: renamed from R1; value 1K -> 50K
- R5: value 1K -> 27R
- Y1: value Crystal -> 12MHz
- renumbered C10 to C1, C1 to C14, C2 to C15, C3 to C16, C11 to C2, C7 to C20, C8 to C21, C9 to C22, J5 to J3, J6 to J5, J7 to J6, R6 to R1, R8 to R3, U5 to U1, U4 to U2, U2 to U5, U3 to U6, U1 to U7
Connections:
- net EXT_3V is gone; now on net +5VD: C21.1, U5.6 (VOUT)
- net EXT_3V_EN is gone; now on net EXT_5V_EN: U5.3 (EN)
- net EXT_3V_FLT is gone; now on net EXT_5V_FLT: U5.4 (FAULT)
- net EXT_5V is gone; now on net VBUS: C20.1, U7.6 (VOUT)
- net PICO_PWR is gone; now on net VDD: C22.1, U6.6 (VOUT)
- net PICO_PWR_EN is gone; now on net VDD_EN: U6.3 (EN)
- net PICO_PWR_FLT is gone; now on net VDD_FLT: U6.4 (FAULT)
- net +3.3V: now also J4.22 (Pin_22), R17.1, R18.1, R19.1, R20.1, TP2.1; no longer C15.2, C18.2, U5.1 (VIN)
- net +5V: now also C15.2, C18.2, U5.1 (VIN), TP3.1
- net EXT_5V_EN: now also J1.42 (GPIO40); no longer U7.3 (EN)
- net EXT_5V_FLT: now also J1.40 (GPIO39), R18.2; no longer U7.4 (FAULT)
- net GND: now also C1.2, C2.2, C6.2, J2.23 (Pin_23), J2.24 (Pin_24), J2.5 (Pin_5), J2.6 (Pin_6), J3.A1 (GND), U1.4 (GND), U1.9 (EP), U2.19 (TESTEN), U2.57 (GND), C10.2, C11.2, C12.2, C13.2, C3.2, C4.2, C5.2, C7.2, C8.2, C9.2, J4.1 (Pin_1), J4.10 (Pin_10), J4.13 (Pin_13), J4.16 (Pin_16), J4.19 (Pin_19), J4.4 (Pin_4), J4.7 (Pin_7), TP1.1, U3.2 (GND), U4.2 (GND)
- net at R3.1: now also C2.1, Y1.2
- net at R3.2: now also U2.21 (XOUT)
- net VDD: now reaches R2.1
- net VDD: now also C6.1, J2.21 (Pin_21), J2.22 (Pin_22), J2.3 (Pin_3), J2.4 (Pin_4), U1.8 (VCC), U2.1 (IOVDD), U2.10 (IOVDD), U2.22 (IOVDD), U2.33 (IOVDD), U2.42 (IOVDD), U2.43 (ADC_AVDD), U2.44 (VREG_IN), U2.48 (USB_VDD), U2.49 (IOVDD), C10.1, C11.1, C12.1, C13.1, C7.1, C8.1, C9.1, R14.2, U3.5 (VBUS)
- net at R2.2: now also R1.2, U1.1 (~{CS}), U2.56 (QSPI_SS)
- net +5VD: now reaches J2.1 (Pin_1)
- net +5VD: now also J2.2 (Pin_2)
- net PICO_IO14: now reaches J2.10 (Pin_10)
- net PICO_IO14: now also U2.17 (GPIO14)
- net PICO_IO9: now reaches J2.11 (Pin_11)
- net PICO_IO9: now also U2.12 (GPIO9)
- net PICO_IO13: now reaches J2.12 (Pin_12)
- net PICO_IO13: now also U2.16 (GPIO13)
- net PICO_IO8: now reaches J2.13 (Pin_13)
- net PICO_IO8: now also U2.11 (GPIO8)
- net PICO_IO12: now reaches J2.14 (Pin_14)
- net PICO_IO12: now also U2.15 (GPIO12)
- net PICO_IO27: now reaches J2.15 (Pin_15)
- net PICO_IO27: now also U2.38 (GPIO26_ADC0)
- net PICO_IO29: now reaches J2.16 (Pin_16)
- net PICO_IO29: now also U2.41 (GPIO29_ADC3)
- net PICO_IO26: now reaches J2.17 (Pin_17)
- net PICO_IO26: now also U2.39 (GPIO27_ADC1)
- net PICO_IO28: now reaches J2.18 (Pin_18)
- net PICO_IO28: now also U2.40 (GPIO28_ADC2)
- net at J2.19 (Pin_19): now also U3.4 (I/O2)
- net at J2.20 (Pin_20): now also U3.6 (I/O1)
- net PICO_IO3: now reaches J2.25 (Pin_25)
- net PICO_IO3: now also U2.5 (GPIO3)
- net PICO_IO7: now reaches J2.26 (Pin_26)
- net PICO_IO7: now also U2.9 (GPIO7)
- net PICO_IO2: now reaches J2.27 (Pin_27)
- net PICO_IO2: now also U2.4 (GPIO2)
- net PICO_IO6: now reaches J2.28 (Pin_28)
- net PICO_IO6: now also U2.8 (GPIO6)
- net PICO_IO1: now reaches J2.29 (Pin_29)
- net PICO_IO1: now also U2.3 (GPIO1)
- net PICO_IO5: now reaches J2.30 (Pin_30)
- net PICO_IO5: now also U2.7 (GPIO5)
- net PICO_IO0: now reaches J2.31 (Pin_31)
- net PICO_IO0: now also U2.2 (GPIO0)
- net PICO_IO4: now reaches J2.32 (Pin_32)
- net PICO_IO4: now also U2.6 (GPIO4)
- net PICO_IO11: now reaches J2.7 (Pin_7)
- net PICO_IO11: now also U2.14 (GPIO11)
- net PICO_IO15: now reaches J2.8 (Pin_8)
- net PICO_IO15: now also U2.18 (GPIO15)
- net PICO_IO10: now reaches J2.9 (Pin_9)
- net PICO_IO10: now also U2.13 (GPIO10)
- net PICO_USB_DN: now reaches R5.1
- net PICO_USB_DN: now also J1.15 (USB4_DM), TP8.1
- net at R5.2: now also U2.46 (USB_DM)
- net VBUS: now reaches J3.A4 (VBUS), J3.A9 (VBUS)
- net VBUS: now also R16.1, R15.1, U4.5 (VBUS)
- net at J3.A5 (CC1): now also R16.2
- net at J3.A6 (D+): now also J3.B6 (D+), U4.4 (I/O2)
- net at J3.A7 (D-): now also J3.B7 (D-), U4.6 (I/O1)
- net at J3.B5 (CC2): now also R15.2
- net at U1.2 (DO(IO1)): now also U2.55 (QSPI_SD1)
- net at U1.3 (IO2): now also U2.54 (QSPI_SD2)
- net at U1.5 (DI(IO0)): now also U2.53 (QSPI_SD0)
- net at U1.6 (CLK): now also U2.52 (QSPI_SCLK)
- net at U1.7 (IO3): now also U2.51 (QSPI_SD3)
- net SPK_RP: now reaches J6.1 (P1)
- net SPK_RP: now also J1.14 (SPK_RP), J6.3 (P2)
- net SPK_RN: now reaches J6.2 (N1)
- net SPK_RN: now also J1.16 (SPK_RN), J6.4 (N2)
- net SPK_LP: now reaches J5.1 (P1)
- net SPK_LP: now also J1.1 (SPK_LP), J5.3 (P2)
- net SPK_LN: now reaches J5.2 (N1)
- net SPK_LN: now also J1.3 (SPK_LN), J5.4 (N2)
- net at C1.1: now also U2.20 (XIN), Y1.1
- net PICO_USB_DP: now reaches J1.13 (USB4_DP)
- net PICO_USB_DP: now also R4.1, TP7.1
- net at J1.18 (GPIO28): now also R6.1
- net at J1.20 (GPIO29): now also R7.1
- net VBUS_FLT: now reaches J1.22 (GPIO30)
- net VBUS_FLT: now also U7.4 (FAULT), R20.2
- net CAM_DP3: now reaches J1.23 (CAM_DP3)
- net CAM_DP3: now also J4.15 (Pin_15)
- net VBUS_EN: now reaches J1.24 (GPIO31)
- net VBUS_EN: now also U7.3 (EN), R17.2
- net CAM_DN3: now reaches J1.25 (CAM_DN3)
- net CAM_DN3: now also J4.14 (Pin_14)
- net UART_TX: now reaches J1.26 (GPIO32)
- net UART_TX: now also R13.2
- net UART_RX: now reaches J1.28 (GPIO33)
- net UART_RX: now also R12.2
- net CAM_DP2: now reaches J1.29 (CAM_DP2)
- net CAM_DP2: now also J4.12 (Pin_12)
- net CAM_DN2: now reaches J1.31 (CAM_DN2)
- net CAM_DN2: now also J4.11 (Pin_11)
- net VDD_FLT: now reaches J1.32 (GPIO35)
- net VDD_FLT: now also R19.2
- net VDD_EN: now reaches J1.34 (GPIO36)
- net VDD_EN: now also TP4.1
- net CAM_CP: now reaches J1.35 (CAM_CP)
- net CAM_CP: now also J4.9 (Pin_9)
- net PICO_BOOT: now reaches J1.36 (GPIO37)
- net PICO_BOOT: now also R1.1, TP6.1
- net CAM_CN: now reaches J1.37 (CAM_CN)
- net CAM_CN: now also J4.8 (Pin_8)
- net PICO_RUN: now reaches J1.38 (GPIO38)
- net PICO_RUN: now also U2.26 (RUN), TP5.1
- net CAM_DP1: now reaches J1.41 (CAM_DP1)
- net CAM_DP1: now also J4.6 (Pin_6)
- net CAM_DN1: now reaches J1.43 (CAM_DN1)
- net CAM_DN1: now also J4.5 (Pin_5)
- net CAM_EN: now reaches J1.46 (GPIO42)
- net CAM_EN: now also J4.17 (Pin_17)
- net CAM_DP0: now reaches J1.47 (CAM_DP0)
- net CAM_DP0: now also J4.3 (Pin_3)
- net CAM_LED: now reaches J1.48 (GPIO43)
- net CAM_LED: now also J4.18 (Pin_18)
- net CAM_DN0: now reaches J1.49 (CAM_DN0)
- net CAM_DN0: now also J4.2 (Pin_2)
- net at J1.50 (GPIO44): now also R8.1
- net at J1.52 (GPIO45): now also R9.1
- net USB_DP: now reaches J1.7 (USB3_DP)
- net USB_DP: now also U4.3 (I/O2)
- net USB_DN: now reaches J1.9 (USB3_DM)
- net USB_DN: now also U4.1 (I/O1)
- net at U2.23 (DVDD), U2.50 (DVDD): now also U2.45 (VREG_VOUT), C3.1, C4.1, C5.1
- net at U2.27 (GPIO16): now also R10.1
- net at U2.28 (GPIO17): now also R11.1
- net at U2.31 (GPIO20): now also R12.1
- net at U2.32 (GPIO21): now also R13.1
- net LED: now reaches U2.37 (GPIO25)
- net LED: now also D1.1 (K)
- net at U2.47 (USB_DP): now also R4.2
- new net: D1.2 (A), R14.1
- new net I2C_SCL: J4.20 (Pin_20), R11.2, R7.2, R9.2, U3.1 (I/O1)
- new net I2C_SDA: J4.21 (Pin_21), R10.2, R6.2, R8.2, U3.3 (I/O2)
- no-connect marks 10 -> 14
Other:
- company: (none) -> vitaly.codes
- title: (none) -> uPico
- moved on the sheet: C1, C14, C15, C16, C17, C18, C19, C2, C20, C21, C22, C6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

Commit message: aux routing
Parts:
- added R15, R16: DNP, Resistor_SMD:R_0402_1005Metric, symbol Device:R
- C1, C10, C11, C12, C13, C17, C18, C19, C2, C3, C4, C5, C6, C7, C8, C9: footprint Capacitor_SMD:C_0402_1005Metric_Pad0.74x0.62mm_HandSolder -> Capacitor_SMD:C_0402_1005Metric
- D1: footprint LED_SMD:LED_0603_1608Metric -> LED_THT:LED_SideEmitter_Rectangular_W4.5mm_H1.6mm
- J1: footprint @upico:uConsoleExt -> @upico:ext
- R1, R2, R3, R4, R5, R8, R9: footprint Resistor_SMD:R_0402_1005Metric_Pad0.72x0.64mm_HandSolder -> Resistor_SMD:R_0402_1005Metric
- R10, R11: value DNP -> 2.2K; footprint Resistor_SMD:R_0402_1005Metric_Pad0.72x0.64mm_HandSolder -> Resistor_SMD:R_0402_1005Metric
- R12: renamed from R14; footprint Resistor_SMD:R_0402_1005Metric_Pad0.72x0.64mm_HandSolder -> Resistor_SMD:R_0402_1005Metric
- R13: renamed from R12; footprint Resistor_SMD:R_0402_1005Metric_Pad0.72x0.64mm_HandSolder -> Resistor_SMD:R_0402_1005Metric
- R14: renamed from R13; footprint Resistor_SMD:R_0402_1005Metric_Pad0.72x0.64mm_HandSolder -> Resistor_SMD:R_0402_1005Metric
- R17: renamed from R15; footprint Resistor_SMD:R_0402_1005Metric_Pad0.72x0.64mm_HandSolder -> Resistor_SMD:R_0402_1005Metric
- R18: renamed from R16; footprint Resistor_SMD:R_0402_1005Metric_Pad0.72x0.64mm_HandSolder -> Resistor_SMD:R_0402_1005Metric
- R19: renamed from R17; footprint Resistor_SMD:R_0402_1005Metric_Pad0.72x0.64mm_HandSolder -> Resistor_SMD:R_0402_1005Metric
- R20: renamed from R18; footprint Resistor_SMD:R_0402_1005Metric_Pad0.72x0.64mm_HandSolder -> Resistor_SMD:R_0402_1005Metric
- R21: renamed from R19; footprint Resistor_SMD:R_0402_1005Metric_Pad0.72x0.64mm_HandSolder -> Resistor_SMD:R_0402_1005Metric
- R22: renamed from R20; footprint Resistor_SMD:R_0402_1005Metric_Pad0.72x0.64mm_HandSolder -> Resistor_SMD:R_0402_1005Metric
- R23: renamed from R21; footprint Resistor_SMD:R_0402_1005Metric_Pad0.72x0.64mm_HandSolder -> Resistor_SMD:R_0402_1005Metric
- R24: renamed from R22; footprint Resistor_SMD:R_0402_1005Metric_Pad0.72x0.64mm_HandSolder -> Resistor_SMD:R_0402_1005Metric
- R25: renamed from R23; footprint Resistor_SMD:R_0402_1005Metric_Pad0.72x0.64mm_HandSolder -> Resistor_SMD:R_0402_1005Metric
- R6, R7: value 0R -> 200R; footprint Resistor_SMD:R_0402_1005Metric_Pad0.72x0.64mm_HandSolder -> Resistor_SMD:R_0402_1005Metric
- U1: value W25Q32JVZP -> W25Q32JV; footprint Package_SON:WSON-8-1EP_6x5mm_P1.27mm_EP3.4x4.3mm -> @upico:USON-8_4x3mm_P0.8mm
Connections:
- net +3.3V: now also R10.1, R11.1
- net I2C_SCL: now also R10.2, R16.2; no longer R11.2
- net I2C_SDA: now also R11.2, R15.2; no longer R10.2
- net VDD: now also D1.2 (A); no longer R12.2
- net at U2.27 (GPIO16): now also R13.1; no longer R10.1
- net at U2.28 (GPIO17): now also R14.1; no longer R11.1
- net at R12.1: now also U2.37 (GPIO25); no longer D1.2 (A)
- net at U2.31 (GPIO20): no longer R13.1
- net at U2.32 (GPIO21): no longer R14.1
- net at U2.29 (GPIO18): now also R15.1
- net at U2.30 (GPIO19): now also R16.1
- net LED: no longer names the net of D1.1 (K)
- net LED: now also R12.2; no longer U2.37 (GPIO25)
- no-connect marks 14 -> 13
Other:
- moved on the sheet: D1, R12, R13, R14, TP1, U3

Commit message: power routing
Parts:
- added C14: 10uF, Capacitor_SMD:C_0603_1608Metric, symbol Device:C
- C5, C6: value 1uF -> 4.7uF
- R12: value 470R -> 510R
- R25: value 50K -> 47K
- R6, R7: value 200R -> DNP
- renumbered C14 to C15, C15 to C16, C16 to C17, C17 to C18, C18 to C19, C19 to C20, C20 to C21, C21 to C22, C22 to C23
Connections:
- net GND: now also C14.1
- net VBUS: now also C14.2

Commit message: control app
Parts:
- H1, H2: footprint MountingHole:MountingHole_2.7mm_M2.5_Pad_Via -> MountingHole:MountingHole_5.3mm_M5
Connections:
- net GND: now also D1.1 (K)
- net PICO_IO0: now also J2.14 (Pin_14); no longer J2.31 (Pin_31)
- net PICO_IO1: now also J2.12 (Pin_12); no longer J2.29 (Pin_29)
- net PICO_IO10: now also J2.28 (Pin_28); no longer J2.9 (Pin_9)
- net PICO_IO11: now also J2.26 (Pin_26); no longer J2.7 (Pin_7)
- net PICO_IO12: now also J2.31 (Pin_31); no longer J2.14 (Pin_14)
- net PICO_IO13: now also J2.29 (Pin_29); no longer J2.12 (Pin_12)
- net PICO_IO14: now also J2.27 (Pin_27); no longer J2.10 (Pin_10)
- net PICO_IO15: now also J2.25 (Pin_25); no longer J2.8 (Pin_8)
- net PICO_IO2: now also J2.10 (Pin_10); no longer J2.27 (Pin_27)
- net PICO_IO26: now also J2.18 (Pin_18); no longer J2.17 (Pin_17)
- net PICO_IO27: now also J2.16 (Pin_16); no longer J2.15 (Pin_15)
- net PICO_IO28: now also J2.17 (Pin_17); no longer J2.18 (Pin_18)
- net PICO_IO29: now also J2.15 (Pin_15); no longer J2.16 (Pin_16)
- net PICO_IO3: now also J2.8 (Pin_8); no longer J2.25 (Pin_25)
- net PICO_IO4: now also J2.13 (Pin_13); no longer J2.32 (Pin_32)
- net PICO_IO5: now also J2.11 (Pin_11); no longer J2.30 (Pin_30)
- net PICO_IO6: now also J2.9 (Pin_9); no longer J2.28 (Pin_28)
- net PICO_IO7: now also J2.7 (Pin_7); no longer J2.26 (Pin_26)
- net PICO_IO8: now also J2.32 (Pin_32); no longer J2.13 (Pin_13)
- net PICO_IO9: now also J2.30 (Pin_30); no longer J2.11 (Pin_11)
- net VDD: no longer D1.2 (A)
- net at U3.4 (I/O2): now also J2.20 (Pin_20); no longer J2.19 (Pin_19)
- net at U3.6 (I/O1): now also J2.19 (Pin_19); no longer J2.20 (Pin_20)
- net at R12.2: now also D1.2 (A); no longer D1.1 (K)
Other:
- moved on the sheet: D1

Commit message: add BOM
Connections:
- no-connect marks 13 -> 12
Changed lines of the file:
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@@
   (no_connect (at 128.27 228.6))
   (no_connect (at 77.47 233.68))
-  (no_connect (at 308.61 30.48))
   (no_connect (at 261.62 81.28))
   (wire (pts (xy 35.56 71.12) (xy 55.88 71.12))

Commit message: change USB connector
Parts:
- removed J3: USB_C, @jb:USB_C_Receptacle_JAE_DX07S016JA3R1500, symbol @jb:USB_C_Receptacle_USB2.0
- removed R13, R14: DNP, Resistor_SMD:R_0402_1005Metric, symbol Device:R
- added J3: USB_C_Receptacle_USB2.0, Connector_USB:USB_C_Receptacle_HRO_TYPE-C-31-M-12, symbol Connector:USB_C_Receptacle_USB2.0
- renumbered R15 to R12, R16 to R13, R12 to R14, R17 to R15, R18 to R16, R19 to R17, R20 to R18, R21 to R19, R22 to R20, R23 to R21, R24 to R22, R25 to R23
Connections:
- net GND: now also J3.A1 (GND), J3.A12 (GND), J3.B1 (GND), J3.B12 (GND)
- net VBUS: now also J3.A4 (VBUS), J3.A9 (VBUS), J3.B4 (VBUS), J3.B9 (VBUS)
- net at R15.2: now also J3.B5 (CC2)
- net at R16.2: now also J3.A5 (CC1)
- net at U4.4 (I/O2): now also J3.A6 (D+), J3.B6 (D+)
- net at U4.6 (I/O1): now also J3.A7 (D-), J3.B7 (D-)
- net UART_RX: no longer names the net of J1.28 (GPIO33)
- net UART_TX: no longer names the net of J1.26 (GPIO32)
- no-connect marks 12 -> 16
Other:
- moved on the sheet: R12, R13

Commit message: update pcb
Parts:
- C1, C2: PN (none) -> C107002
- C10, C11, C12, C13, C18, C19, C20, C3, C4, C7, C8, C9: PN (none) -> C1525
- C14, C15, C16, C17, C21, C22, C23: PN (none) -> C96446
- C5, C6: PN (none) -> C23733
- D1: now left out of the parts list
- J2: PN (none) -> C2897436
- J3: PN (none) -> C165948
- J4: PN (none) -> C11091; now left out of the parts list
- R1, R3: PN (none) -> C11702
- R10, R11: PN (none) -> C25879
- R14: PN (none) -> C25123
- R15, R16: PN (none) -> C114756
- R17, R18, R19, R20: PN (none) -> C25744
- R21, R22: PN (none) -> C25741
- R23: value 47K -> 56K; PN (none) -> C114756
- R4, R5: PN (none) -> C226392
- U1: value W25Q32JV -> W25Q32JVUX; footprint @upico:USON-8_4x3mm_P0.8mm -> @upico:USON-8_2x3mm_P0.5mm; PN (none) -> C2843335
- U2: PN (none) -> C2040
- U3, U4: PN (none) -> C15999
- U5: value AP22652_3x -> AP22652
- U6, U7: value AP22652_3x -> AP22652; PN (none) -> C2158038
- Y1: PN (none) -> C3035208
Other:
- note added: "Ilim = 30321 / R 100K => 300mA"
- note added: "Ilim = 30321 / R 56K => 540mA"
